Commit message: Updated Robot URDF's with success Launch

File: cable_robot_ws/src/cable_robot_description/install/cable_robot_description/share/cable_robot_description/urdf/cable_robot.urdf.xacro (robot description, xacro)
@@ -1,25 +1,47 @@
 <?xml version="1.0"?>
 <robot xmlns:xacro="http://www.ros.org/wiki/xacro" name="cable_robot">
+    <!-- Include component macros -->
+    <xacro:include filename="$(find cable_robot_description)/urdf/components/frame.urdf.xacro"/>
+    <xacro:include filename="$(find cable_robot_description)/urdf/components/cable.urdf.xacro"/>
+    <xacro:include filename="$(find cable_robot_description)/urdf/components/winch.urdf.xacro"/>
+    <!-- Define robot properties -->
+    <xacro:property name="frame_height" value="2.0"/>
+    <xacro:property name="frame_width" value="2.0"/>
+    <xacro:property name="frame_length" value="2.0"/>
+    <xacro:property name="drum_radius" value="0.05"/>
+    <xacro:property name="drum_length" value="0.1"/>
+    <xacro:property name="winch_gear_ratio" value="50.0"/>
+    <xacro:property name="cable_radius" value="0.002"/>
+    <xacro:property name="cable_max_length" value="3.0"/>
+    <xacro:property name="cable_max_tension" value="1000.0"/>
+    <xacro:property name="cable_max_velocity" value="1.0"/>
+    <!-- Base Link -->
     <link name="base_link">
         <visual>
+            <origin xyz="0 0 0" rpy="0 0 0"/>
             <geometry>
-                <box size="0.5 0.5 0.1"/>
+                <box size="0.1 0.1 0.001"/>
             </geometry>
-            <material name="blue">
-                <color rgba="0 0 1 1"/>
+            <material name="base_material">
+                <color rgba="0.5 0.5 0.5 1"/>
             </material>
         </visual>
         <collision>
+            <origin xyz="0 0 0" rpy="0 0 0"/>
             <geometry>
-                <box size="0.5 0.5 0.1"/>
+                <box size="0.1 0.1 0.001"/>
             </geometry>
         </collision>
         <inertial>
+            <origin xyz="0 0 0" rpy="0 0 0"/>
             <mass value="1.0"/>
-            <inertia ixx="0.0416" ixy="0" ixz="0" iyy="0.0416" iyz="0" izz="0.0833"/>
+            <inertia ixx="0.001" ixy="0" ixz="0"
+                     iyy="0.001" iyz="0"
+                     izz="0.001"/>
         </inertial>
     </link>
-    <gazebo reference="base_link">
-        <material>Gazebo/Blue</material>
-    </gazebo>
+    <!-- Frame -->
+    <xacro:complete_frame parent="base_link">
+        <origin xyz="0 0 0.05" rpy="0 0 0"/>
+    </xacro:complete_frame>
 </robot>

File: cable_robot_ws/src/cable_robot_description/install/cable_robot_description/share/cable_robot_description/urdf/components/cable.urdf.xacro (robot description, xacro)
@@ -2,5 +2,5 @@
 <robot xmlns:xacro="http://www.ros.org/wiki/xacro">
     <!-- Cable macro for CDPR -->
-    <xacro:macro name="cable_macro" params="prefix base_point platform_point parent child">
+    <xacro:macro name="cable_macro" params="prefix parent child base_point:='0 0 0' platform_point:='0 0 0'">
         <!-- Virtual link for cable -->
         <link name="${prefix}_link">

File: cable_robot_ws/src/cable_robot_description/install/cable_robot_description/share/cable_robot_description/urdf/components/frame.urdf.xacro (robot description, xacro)
@@ -2,5 +2,5 @@
 <robot xmlns:xacro="http://www.ros.org/wiki/xacro">
     <!-- Include the pillar macro -->
-    <xacro:include filename="$(find CDPRX)/urdf/components/pillar.urdf.xacro"/>
+    <xacro:include filename="$(find cable_robot_description)/urdf/components/frame_pillar.urdf.xacro"/>
     <!-- Complete frame macro -->
     <xacro:macro name="complete_frame" params="parent *origin">
@@ -21,14 +21,10 @@
         <!-- Front right pillar -->
         <xacro:property name="fr_heights" value="${[frame_height * 0.8, frame_height * 0.6]}"/>
-        <xacro:property name="fr_angles" value="${[pi/4, pi/4]}"/>
         <!-- Front left pillar -->
         <xacro:property name="fl_heights" value="${[frame_height * 0.8, frame_height * 0.6]}"/>
-        <xacro:property name="fl_angles" value="${[-pi/4, -pi/4]}"/>
         <!-- Back right pillar -->
         <xacro:property name="br_heights" value="${[frame_height * 0.8, frame_height * 0.6]}"/>
-        <xacro:property name="br_angles" value="${[3*pi/4, 3*pi/4]}"/>
         <!-- Back left pillar -->
         <xacro:property name="bl_heights" value="${[frame_height * 0.8, frame_height * 0.6]}"/>
-        <xacro:property name="bl_angles" value="${[-3*pi/4, -3*pi/4]}"/>
         <!-- Create four pillars -->
         <xacro:frame_pillar prefix="pillar_front_right"
@@ -36,24 +32,24 @@
                            position_x="${frame_length/2}"
                            position_y="${frame_width/2}"
-                           outlet_heights="${fr_heights}"
-                           outlet_angles="${fr_angles}"/>
+                           height="${frame_height}"
+                           outlet_heights="${fr_heights}"/>
         <xacro:frame_pillar prefix="pillar_front_left"
                            parent="frame_center"
                            position_x="${frame_length/2}"
                            position_y="${-frame_width/2}"
-                           outlet_heights="${fl_heights}"
-                           outlet_angles="${fl_angles}"/>
+                           height="${frame_height}"
+                           outlet_heights="${fl_heights}"/>
         <xacro:frame_pillar prefix="pillar_back_right"
                            parent="frame_center"
                            position_x="${-frame_length/2}"
                            position_y="${frame_width/2}"
-                           outlet_heights="${br_heights}"
-                           outlet_angles="${br_angles}"/>
+                           height="${frame_height}"
+                           outlet_heights="${br_heights}"/>
         <xacro:frame_pillar prefix="pillar_back_left"
                            parent="frame_center"
                            position_x="${-frame_length/2}"
                            position_y="${-frame_width/2}"
-                           outlet_heights="${bl_heights}"
-                           outlet_angles="${bl_angles}"/>
+                           height="${frame_height}"
+                           outlet_heights="${bl_heights}"/>
     </xacro:macro>
 </robot>

File: cable_robot_ws/src/cable_robot_description/urdf/components/frame_pillar.urdf.xacro (robot description, xacro)
@@ -1,8 +1,21 @@
 <?xml version="1.0"?>
 <robot xmlns:xacro="http://www.ros.org/wiki/xacro">
-    <!-- Include pillar properties -->
-    <xacro:include filename="$(find CDPRX)/urdf/properties/pillar_properties.xacro"/>
+    <!-- Pillar properties -->
+    <xacro:property name="pillar_base_length" value="0.3"/>
+    <xacro:property name="pillar_base_width" value="0.3"/>
+    <xacro:property name="pillar_base_height" value="0.05"/>
+    <xacro:property name="pillar_width" value="0.1"/>
+    <xacro:property name="pillar_length" value="0.1"/>
+    <xacro:property name="base_mass" value="5.0"/>
+    <xacro:property name="pillar_mass" value="10.0"/>
+    <xacro:property name="outlet_radius" value="0.02"/>
+    <xacro:property name="outlet_offset" value="0.02"/>
+    <!-- Calculate inertias -->
+    <xacro:property name="base_ixx" value="${(base_mass/12.0) * (pillar_base_width*pillar_base_width + pillar_base_height*pillar_base_height)}"/>
+    <xacro:property name="base_iyy" value="${(base_mass/12.0) * (pillar_base_length*pillar_base_length + pillar_base_height*pillar_base_height)}"/>
+    <xacro:property name="pillar_ixx" value="${(pillar_mass/12.0) * (pillar_width*pillar_width)}"/>
+    <xacro:property name="pillar_iyy" value="${(pillar_mass/12.0) * (pillar_length*pillar_length)}"/>
     <!-- Single pillar macro -->
-    <xacro:macro name="frame_pillar" params="prefix parent position_x position_y height *origin outlet_heights:=^">
+    <xacro:macro name="frame_pillar" params="prefix parent position_x position_y height outlet_heights:=^">
         <!-- Base plate -->
         <link name="${prefix}_base">
@@ -57,5 +70,5 @@
                     ixx="${pillar_ixx}" ixy="0" ixz="0"
                     iyy="${pillar_iyy}" iyz="0"
-                    izz="${(pillar_mass/12.0) * (pillar_width*pillar_width + pillar_length*pillar_length)}"/>
+                    izz="${pillar_mass/12.0 * (pillar_width*pillar_width + pillar_length*pillar_length)}"/>
             </inertial>
         </link>
