Commit message: Experimentation with Gazebo CDPRs

File: cable_robot_ws/src/cable_robot_description/urdf/cable_robot.urdf.xacro (robot description, xacro)
@@ -16,32 +16,120 @@
     <xacro:property name="cable_max_tension" value="1000.0"/>
     <xacro:property name="cable_max_velocity" value="1.0"/>
-    <!-- Base Link -->
-    <link name="base_link">
-        <visual>
-            <origin xyz="0 0 0" rpy="0 0 0"/>
-            <geometry>
-                <box size="0.1 0.1 0.001"/>
-            </geometry>
-            <material name="base_material">
-                <color rgba="0.5 0.5 0.5 1"/>
-            </material>
-        </visual>
-        <collision>
-            <origin xyz="0 0 0" rpy="0 0 0"/>
-            <geometry>
-                <box size="0.1 0.1 0.001"/>
-            </geometry>
-        </collision>
+    <!-- World link -->
+    <link name="world"/>
+    <!-- Base link with dummy link to handle KDL -->
+    <link name="dummy_base">
         <inertial>
             <origin xyz="0 0 0" rpy="0 0 0"/>
-            <mass value="1.0"/>
-            <inertia ixx="0.001" ixy="0" ixz="0"
-                     iyy="0.001" iyz="0"
-                     izz="0.001"/>
+            <mass value="0.0001"/>
+            <inertia ixx="0.0001" ixy="0" ixz="0"
+                     iyy="0.0001" iyz="0"
+                     izz="0.0001"/>
         </inertial>
     </link>
-    <!-- Frame -->
-    <xacro:complete_frame parent="base_link">
+    <joint name="world_to_dummy" type="fixed">
+        <parent link="world"/>
+        <child link="dummy_base"/>
+        <origin xyz="0 0 0" rpy="0 0 0"/>
+    </joint>
+    <link name="base_link"/>
+    <joint name="dummy_to_base" type="fixed">
+        <parent link="dummy_base"/>
+        <child link="base_link"/>
+        <origin xyz="0 0 0" rpy="0 0 0"/>
+    </joint>
+    <!-- Modular frame -->
+    <xacro:modular_frame parent="base_link">
         <origin xyz="0 0 0.05" rpy="0 0 0"/>
-    </xacro:complete_frame>
+    </xacro:modular_frame>
+    <!-- Independent pillars -->
+    <xacro:modular_pillar name="pillar_front_right"
+                          parent="base_link"
+                          position_x="${frame_length/2}"
+                          position_y="${frame_width/2}"
+                          height="${frame_height}"
+                          outlet_height="${frame_height * 0.8}"/>
+    <xacro:modular_pillar name="pillar_front_left"
+                          parent="base_link"
+                          position_x="${frame_length/2}"
+                          position_y="${-frame_width/2}"
+                          height="${frame_height}"
+                          outlet_height="${frame_height * 0.8}"/>
+    <xacro:modular_pillar name="pillar_back_right"
+                          parent="base_link"
+                          position_x="${-frame_length/2}"
+                          position_y="${frame_width/2}"
+                          height="${frame_height}"
+                          outlet_height="${frame_height * 0.8}"/>
+    <xacro:modular_pillar name="pillar_back_left"
+                          parent="base_link"
+                          position_x="${-frame_length/2}"
+                          position_y="${-frame_width/2}"
+                          height="${frame_height}"
+                          outlet_height="${frame_height * 0.8}"/>
+    <!-- Winch systems -->
+    <xacro:modular_winch name="winch_fr"
+                         parent="pillar_front_right_outlet_mount"
+                         drum_radius="${drum_radius}"
+                         drum_length="${drum_length}"
+                         gear_ratio="${winch_gear_ratio}">
+        <origin xyz="0.1 0 0" rpy="0 ${pi/2} 0"/>
+    </xacro:modular_winch>
+    <xacro:modular_winch name="winch_fl"
+                         parent="pillar_front_left_outlet_mount"
+                         drum_radius="${drum_radius}"
+                         drum_length="${drum_length}"
+                         gear_ratio="${winch_gear_ratio}">
+        <origin xyz="0.1 0 0" rpy="0 ${pi/2} 0"/>
+    </xacro:modular_winch>
+    <xacro:modular_winch name="winch_br"
+                         parent="pillar_back_right_outlet_mount"
+                         drum_radius="${drum_radius}"
+                         drum_length="${drum_length}"
+                         gear_ratio="${winch_gear_ratio}">
+        <origin xyz="-0.1 0 0" rpy="0 ${pi/2} ${pi}"/>
+    </xacro:modular_winch>
+    <xacro:modular_winch name="winch_bl"
+                         parent="pillar_back_left_outlet_mount"
+                         drum_radius="${drum_radius}"
+                         drum_length="${drum_length}"
+                         gear_ratio="${winch_gear_ratio}">
+        <origin xyz="-0.1 0 0" rpy="0 ${pi/2} ${pi}"/>
+    </xacro:modular_winch>
+    <!-- Cable systems -->
+    <xacro:modular_cable name="cable_fr"
+                        parent_mount="winch_fr_output_mount"
+                        child_mount="platform_base"
+                        radius="${cable_radius}"
+                        max_length="${cable_max_length}"
+                        max_tension="${cable_max_tension}"
+                        max_velocity="${cable_max_velocity}"/>
+    <xacro:modular_cable name="cable_fl"
+                        parent_mount="winch_fl_output_mount"
+                        child_mount="platform_base"
+                        radius="${cable_radius}"
+                        max_length="${cable_max_length}"
+                        max_tension="${cable_max_tension}"
+                        max_velocity="${cable_max_velocity}"/>
+    <xacro:modular_cable name="cable_br"
+                        parent_mount="winch_br_output_mount"
+                        child_mount="platform_base"
+                        radius="${cable_radius}"
+                        max_length="${cable_max_length}"
+                        max_tension="${cable_max_tension}"
+                        max_velocity="${cable_max_velocity}"/>
+    <xacro:modular_cable name="cable_bl"
+                        parent_mount="winch_bl_output_mount"
+                        child_mount="platform_base"
+                        radius="${cable_radius}"
+                        max_length="${cable_max_length}"
+                        max_tension="${cable_max_tension}"
+                        max_velocity="${cable_max_velocity}"/>
+    <!-- Gazebo plugin for the platform -->
+    <gazebo>
+        <plugin name="gazebo_ros_control" filename="libgazebo_ros_control.so">
+            <robotNamespace>/cable_robot</robotNamespace>
+            <robotSimType>gazebo_ros_control/DefaultRobotHWSim</robotSimType>
+        </plugin>
+    </gazebo>
 </robot>

File: cable_robot_ws/src/cable_robot_description/urdf/components/cable.urdf.xacro (robot description, xacro)
@@ -1,65 +1,57 @@
 <?xml version="1.0"?>
 <robot xmlns:xacro="http://www.ros.org/wiki/xacro">
-    <!-- Cable macro for CDPR -->
-    <xacro:macro name="cable_macro" params="prefix parent child base_point:='0 0 0' platform_point:='0 0 0'">
-        <!-- Virtual link for cable -->
-        <link name="${prefix}_link">
+    <!-- Modular cable system macro -->
+    <xacro:macro name="modular_cable" params="name parent_mount child_mount radius max_length max_tension max_velocity">
+        <!-- Cable link -->
+        <link name="${name}_link">
             <visual>
                 <geometry>
-                    <cylinder radius="${cable_radius}" length="${cable_max_length}"/>
+                    <cylinder radius="${radius}" length="0.1"/>
                 </geometry>
                 <material name="cable_material">
-                    <color rgba="0.8 0.8 0.8 1"/>
+                    <color rgba="0.1 0.1 0.1 1"/>
                 </material>
             </visual>
+            <collision>
+                <geometry>
+                    <cylinder radius="${radius}" length="0.1"/>
+                </geometry>
+            </collision>
             <inertial>
-                <!-- Near-zero mass for cable -->
-                <mass value="0.001"/>
-                <inertia ixx="0.001" ixy="0" ixz="0" iyy="0.001" iyz="0" izz="0.001"/>
+                <mass value="0.1"/>
+                <inertia ixx="0.001" ixy="0" ixz="0"
+                         iyy="0.001" iyz="0"
+                         izz="0.001"/>
             </inertial>
         </link>
-        <!-- Universal joint at base -->
-        <joint name="${prefix}_base_joint" type="universal">
-            <parent link="${parent}"/>
-            <child link="${prefix}_link"/>
-            <origin xyz="${base_point}" rpy="0 0 0"/>
-            <axis xyz="1 0 0"/>
-            <axis2 xyz="0 1 0"/>
-            <dynamics damping="0.1" friction="0.1"/>
+        <!-- Cable attachment joints -->
+        <joint name="${name}_winch_joint" type="fixed">
+            <parent link="${parent_mount}"/>
+            <child link="${name}_link"/>
+            <origin xyz="0 0 0" rpy="0 0 0"/>
         </joint>
-        <!-- Prismatic joint for cable extension -->
-        <joint name="${prefix}_extension" type="prismatic">
-            <parent link="${prefix}_link"/>
-            <child link="${prefix}_end_link"/>
+        <joint name="${name}_platform_joint" type="fixed">
+            <parent link="${name}_link"/>
+            <child link="${child_mount}"/>
             <origin xyz="0 0 0" rpy="0 0 0"/>
-            <axis xyz="0 0 1"/>
-            <limit lower="0" upper="${cable_max_length}"
-                   effort="${cable_max_tension}" velocity="${cable_max_velocity}"/>
-            <dynamics damping="0.1" friction="0.1"/>
         </joint>
-        <!-- Virtual end link -->
-        <link name="${prefix}_end_link">
-            <inertial>
-                <mass value="0.001"/>
-                <inertia ixx="0.001" ixy="0" ixz="0" iyy="0.001" iyz="0" izz="0.001"/>
-            </inertial>
-        </link>
-        <!-- Spherical joint at platform -->
-        <joint name="${prefix}_platform_joint" type="spherical">
-            <parent link="${prefix}_end_link"/>
-            <child link="${child}"/>
-            <origin xyz="${platform_point}" rpy="0 0 0"/>
-            <dynamics damping="0.1" friction="0.1"/>
-        </joint>
-        <!-- Add transmission for actuation -->
-        <transmission name="${prefix}_trans">
-            <type>transmission_interface/SimpleTransmission</type>
-            <joint name="${prefix}_extension">
-                <hardwareInterface>hardware_interface/EffortJointInterface</hardwareInterface>
-            </joint>
-            <actuator name="${prefix}_motor">
-                <mechanicalReduction>1</mechanicalReduction>
-            </actuator>
-        </transmission>
+        <!-- Gazebo-specific properties -->
+        <gazebo reference="${name}_link">
+            <material>Gazebo/Black</material>
+            <mu1>0.5</mu1>
+            <mu2>0.5</mu2>
+        </gazebo>
+        <!-- Cable plugin -->
+        <gazebo>
+            <plugin name="${name}_plugin" filename="libgazebo_ros_cable.so">
+                <robotNamespace>/cable_robot</robotNamespace>
+                <linkName>${name}_link</linkName>
+                <winchJointName>${name}_winch_joint</winchJointName>
+                <platformJointName>${name}_platform_joint</platformJointName>
+                <maxLength>${max_length}</maxLength>
+                <maxTension>${max_tension}</maxTension>
+                <maxVelocity>${max_velocity}</maxVelocity>
+            </plugin>
+        </gazebo>
     </xacro:macro>
 </robot>

File: cable_robot_ws/src/cable_robot_description/urdf/components/frame.urdf.xacro (robot description, xacro)
@@ -1,8 +1,128 @@
 <?xml version="1.0"?>
 <robot xmlns:xacro="http://www.ros.org/wiki/xacro">
-    <!-- Include the pillar macro -->
-    <xacro:include filename="$(find cable_robot_description)/urdf/components/frame_pillar.urdf.xacro"/>
-    <!-- Complete frame macro -->
-    <xacro:macro name="complete_frame" params="parent *origin">
+    <!-- Include necessary components -->
+    <xacro:include filename="$(find cable_robot_description)/urdf/components/platform.urdf.xacro"/>
+    <!-- Joint helper macros -->
+    <xacro:macro name="prismatic_joint_link" params="name parent axis">
+        <joint name="platform_${name}" type="prismatic">
+            <parent link="${parent}"/>
+            <child link="platform_${name}"/>
+            <axis xyz="${axis}"/>
+            <limit lower="-${frame_length}" upper="${frame_length}" effort="1000" velocity="1.0"/>
+        </joint>
+        <link name="platform_${name}">
+            <inertial>
+                <mass value="0.1"/>
+                <inertia ixx="0.001" ixy="0" ixz="0"
+                         iyy="0.001" iyz="0"
+                         izz="0.001"/>
+            </inertial>
+        </link>
+    </xacro:macro>
+    <xacro:macro name="revolute_joint_link" params="name parent axis">
+        <joint name="platform_${name}" type="revolute">
+            <parent link="${parent}"/>
+            <child link="platform_${name}"/>
+            <axis xyz="${axis}"/>
+            <limit lower="-${pi}" upper="${pi}" effort="1000" velocity="1.0"/>
+        </joint>
+        <link name="platform_${name}">
+            <inertial>
+                <mass value="0.1"/>
+                <inertia ixx="0.001" ixy="0" ixz="0"
+                         iyy="0.001" iyz="0"
+                         izz="0.001"/>
+            </inertial>
+        </link>
+    </xacro:macro>
+    <!-- Mounting point macro -->
+    <xacro:macro name="cable_mount" params="name parent *origin">
+        <link name="${name}_mount">
+            <visual>
+                <geometry>
+                    <cylinder radius="0.01" length="0.02"/>
+                </geometry>
+                <material name="mount_material">
+                    <color rgba="0.8 0.8 0.8 1"/>
+                </material>
+            </visual>
+            <collision>
+                <geometry>
+                    <cylinder radius="0.01" length="0.02"/>
+                </geometry>
+            </collision>
+            <inertial>
+                <mass value="0.05"/>
+                <inertia ixx="0.001" ixy="0" ixz="0"
+                         iyy="0.001" iyz="0"
+                         izz="0.001"/>
+            </inertial>
+        </link>
+        <joint name="${name}_mount_joint" type="fixed">
+            <parent link="${parent}"/>
+            <child link="${name}_mount"/>
+            <xacro:insert_block name="origin"/>
+        </joint>
+    </xacro:macro>
+    <!-- Individual pillar macro with cable outlet -->
+    <xacro:macro name="modular_pillar" params="name parent position_x position_y height outlet_height">
+        <!-- Pillar base -->
+        <link name="${name}_base">
+            <visual>
+                <geometry>
+                    <box size="0.1 0.1 0.05"/>
+                </geometry>
+            </visual>
+            <collision>
+                <geometry>
+                    <box size="0.1 0.1 0.05"/>
+                </geometry>
+            </collision>
+            <inertial>
+                <mass value="1.0"/>
+                <inertia ixx="0.01" ixy="0" ixz="0"
+                         iyy="0.01" iyz="0"
+                         izz="0.01"/>
+            </inertial>
+        </link>
+        <joint name="${name}_base_joint" type="fixed">
+            <parent link="${parent}"/>
+            <child link="${name}_base"/>
+            <origin xyz="${position_x} ${position_y} 0" rpy="0 0 0"/>
+        </joint>
+        <!-- Pillar column -->
+        <link name="${name}_column">
+            <visual>
+                <geometry>
+                    <cylinder radius="0.05" length="${height}"/>
+                </geometry>
+                <origin xyz="0 0 ${height/2}" rpy="0 0 0"/>
+            </visual>
+            <collision>
+                <geometry>
+                    <cylinder radius="0.05" length="${height}"/>
+                </geometry>
+                <origin xyz="0 0 ${height/2}" rpy="0 0 0"/>
+            </collision>
+            <inertial>
+                <mass value="2.0"/>
+                <origin xyz="0 0 ${height/2}" rpy="0 0 0"/>
+                <inertia ixx="0.1" ixy="0" ixz="0"
+                         iyy="0.1" iyz="0"
+                         izz="0.01"/>
+            </inertial>
+        </link>
+        <joint name="${name}_column_joint" type="fixed">
+            <parent link="${name}_base"/>
+            <child link="${name}_column"/>
+            <origin xyz="0 0 0" rpy="0 0 0"/>
+        </joint>
+        <!-- Cable outlet -->
+        <xacro:cable_mount name="${name}_outlet" parent="${name}_column">
+            <origin xyz="0 0 ${outlet_height}" rpy="0 0 0"/>
+        </xacro:cable_mount>
+    </xacro:macro>
+    <!-- Frame assembly macro -->
+    <xacro:macro name="modular_frame" params="parent *origin">
         <!-- Frame center reference -->
         <link name="frame_center">
@@ -12,4 +132,10 @@
                 </geometry>
             </visual>
+            <inertial>
+                <mass value="0.1"/>
+                <inertia ixx="0.001" ixy="0" ixz="0"
+                         iyy="0.001" iyz="0"
+                         izz="0.001"/>
+            </inertial>
         </link>
         <joint name="frame_center_joint" type="fixed">
@@ -18,38 +144,41 @@
             <xacro:insert_block name="origin"/>
         </joint>
-        <!-- Define outlet configurations for each pillar -->
-        <!-- Front right pillar -->
-        <xacro:property name="fr_heights" value="${[frame_height * 0.8, frame_height * 0.6]}"/>
-        <!-- Front left pillar -->
-        <xacro:property name="fl_heights" value="${[frame_height * 0.8, frame_height * 0.6]}"/>
-        <!-- Back right pillar -->
-        <xacro:property name="br_heights" value="${[frame_height * 0.8, frame_height * 0.6]}"/>
-        <!-- Back left pillar -->
-        <xacro:property name="bl_heights" value="${[frame_height * 0.8, frame_height * 0.6]}"/>
-        <!-- Create four pillars -->
-        <xacro:frame_pillar prefix="pillar_front_right"
-                           parent="frame_center"
-                           position_x="${frame_length/2}"
-                           position_y="${frame_width/2}"
-                           height="${frame_height}"
-                           outlet_heights="${fr_heights}"/>
-        <xacro:frame_pillar prefix="pillar_front_left"
-                           parent="frame_center"
-                           position_x="${frame_length/2}"
-                           position_y="${-frame_width/2}"
-                           height="${frame_height}"
-                           outlet_heights="${fl_heights}"/>
-        <xacro:frame_pillar prefix="pillar_back_right"
-                           parent="frame_center"
-                           position_x="${-frame_length/2}"
-                           position_y="${frame_width/2}"
-                           height="${frame_height}"
-                           outlet_heights="${br_heights}"/>
-        <xacro:frame_pillar prefix="pillar_back_left"
-                           parent="frame_center"
-                           position_x="${-frame_length/2}"
-                           position_y="${-frame_width/2}"
-                           height="${frame_height}"
-                           outlet_heights="${bl_heights}"/>
+        <!-- Platform with 6-DOF joints -->
+        <xacro:platform_6dof parent="frame_center"/>
+    </xacro:macro>
+    <!-- Platform 6-DOF joints macro -->
+    <xacro:macro name="platform_6dof" params="parent">
+        <!-- Create intermediate links and joints for 6-DOF movement -->
+        <xacro:create_platform_chain parent="${parent}"/>
+        <!-- Add the end-effector platform -->
+        <xacro:end_effector_platform parent="platform_base">
+            <origin xyz="0 0 0" rpy="0 0 0"/>
+        </xacro:end_effector_platform>
+    </xacro:macro>
+    <!-- Helper macro to create the 6-DOF joint chain -->
+    <xacro:macro name="create_platform_chain" params="parent">
+        <!-- Same implementation as your original 6-DOF chain,
+             but now in a separate macro for better modularity -->
+        <link name="platform_base">
+            <inertial>
+                <mass value="1.0"/>
+                <inertia ixx="0.1" ixy="0" ixz="0"
+                         iyy="0.1" iyz="0"
+                         izz="0.1"/>
+            </inertial>
+        </link>
+        <!-- X, Y, Z prismatic joints -->
+        <xacro:prismatic_joint_link name="x" parent="${parent}" axis="1 0 0"/>
+        <xacro:prismatic_joint_link name="y" parent="platform_x" axis="0 1 0"/>
+        <xacro:prismatic_joint_link name="z" parent="platform_y" axis="0 0 1"/>
+        <!-- Roll, Pitch, Yaw revolute joints -->
+        <xacro:revolute_joint_link name="roll" parent="platform_z" axis="1 0 0"/>
+        <xacro:revolute_joint_link name="pitch" parent="platform_roll" axis="0 1 0"/>
+        <joint name="platform_yaw" type="revolute">
+            <parent link="platform_pitch"/>
+            <child link="platform_base"/>
+            <axis xyz="0 0 1"/>
+            <limit lower="-${pi}" upper="${pi}" effort="1000" velocity="1.0"/>
+        </joint>
     </xacro:macro>
 </robot>
